File: split-left/output-left/pcbs/pcb-left-rc1--no-smd.kicad_pcb (KiCad board)
At the start: 2 copper layers, 153.9 x 144.5 mm, 86 parts

Commit message: Stopped pth's from being on the silk screen layer and creating drc errors because it was printing the hole into the silkscreen. Also fixed my custom blackpill footprint that created the problem
Other:
- rule pad_to_mask_clearance: 0.05 -> 0.038
Changed lines of the file:
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@@
 	)
 	(setup
-		(pad_to_mask_clearance 0.05)
+		(pad_to_mask_clearance 0.038)
 		(allow_soldermask_bridges_in_footprints no)
 		(pcbplotparams
@@
 			(size 1.7526 1.7526)
 			(drill 1.0922)
-			(layers "*.Cu" "*.SilkS" "*.Mask")
+			(layers "*.Cu" "*.Mask")
 			(remove_unused_layers no)
 			(net 65 "A0")
@@
 			(size 1.7526 1.7526)
 			(drill 1.0922)
-			(layers "*.Cu" "*.SilkS" "*.Mask")
+			(layers "*.Cu" "*.Mask")
 			(remove_unused_layers no)
 			(net 64 "A1")
@@
 			(size 1.7526 1.7526)
 			(drill 1.0922)
-			(layers "*.Cu" "*.SilkS" "*.Mask")
+			(layers "*.Cu" "*.Mask")
 			(remove_unused_layers no)
 			(net 63 "A2")
@@
 			(size 1.7526 1.7526)
 			(drill 1.0922)
-			(layers "*.Cu" "*.SilkS" "*.Mask")
+			(layers "*.Cu" "*.Mask")
 			(remove_unused_layers no)
 			(net 62 "A3")
@@
 			(size 1.7526 1.7526)
 			(drill 1.0922)
-			(layers "*.Cu" "*.SilkS" "*.Mask")
+			(layers "*.Cu" "*.Mask")
 			(remove_unused_layers no)
 			(net 61 "A4")
@@
 			(size 1.7526 1.7526)
 			(drill 1.0922)
-			(layers "*.Cu" "*.SilkS" "*.Mask")
+			(layers "*.Cu" "*.Mask")
 			(remove_unused_layers no)
 			(net 60 "A5")
@@
 			(size 1.7526 1.7526)
 			(drill 1.0922)
-			(layers "*.Cu" "*.SilkS" "*.Mask")
+			(layers "*.Cu" "*.Mask")
 			(remove_unused_layers no)
 			(net 59 "A6")
@@
 			(size 1.7526 1.7526)
 			(drill 1.0922)
-			(layers "*.Cu" "*.SilkS" "*.Mask")
+			(layers "*.Cu" "*.Mask")
 			(remove_unused_layers no)
 			(net 58 "A7")
@@
 			(size 1.7526 1.7526)
 			(drill 1.0922)
-			(layers "*.Cu" "*.SilkS" "*.Mask")
+			(layers "*.Cu" "*.Mask")
 			(remove_unused_layers no)
 			(net 9 "A8")
@@
 			(size 1.7526 1.7526)
 			(drill 1.0922)
-			(layers "*.Cu" "*.SilkS" "*.Mask")
+			(layers "*.Cu" "*.Mask")
 			(remove_unused_layers no)
 			(net 11 "A9")
@@
 			(size 1.7526 1.7526)
 			(drill 1.0922)
-			(layers "*.Cu" "*.SilkS" "*.Mask")
+			(layers "*.Cu" "*.Mask")
 			(remove_unused_layers no)
 			(net 13 "A10")
@@
 			(size 1.7526 1.7526)
 			(drill 1.0922)
-			(layers "*.Cu" "*.SilkS" "*.Mask")
+			(layers "*.Cu" "*.Mask")
 			(remove_unused_layers no)
 			(net 73 "A15")
@@
 			(size 1.7526 1.7526)
 			(drill 1.0922)
-			(layers "*.Cu" "*.SilkS" "*.Mask")
+			(layers "*.Cu" "*.Mask")
 			(remove_unused_layers no)
 			(net 57 "B0")
@@
 			(size 1.7526 1.7526)
 			(drill 1.0922)
-			(layers "*.Cu" "*.SilkS" "*.Mask")
+			(layers "*.Cu" "*.Mask")
 			(remove_unused_layers no)
 			(net 56 "B1")
@@
 			(size 1.7526 1.7526)
 			(drill 1.0922)
-			(layers "*.Cu" "*.SilkS" "*.Mask")
+			(layers "*.Cu" "*.Mask")
 			(remove_unused_layers no)
 			(net 74 "B3")
@@
 			(size 1.7526 1.7526)
 			(drill 1.0922)
-			(layers "*.Cu" "*.SilkS" "*.Mask")
+			(layers "*.Cu" "*.Mask")
 			(remove_unused_layers no)
 			(net 49 "B4")
@@
 			(size 1.7526 1.7526)
 			(drill 1.0922)
-			(layers "*.Cu" "*.SilkS" "*.Mask")
+			(layers "*.Cu" "*.Mask")
 			(remove_unused_layers no)
 			(net 45 "B5")
@@
 			(size 1.7526 1.7526)
 			(drill 1.0922)
-			(layers "*.Cu" "*.SilkS" "*.Mask")
+			(layers "*.Cu" "*.Mask")
 			(remove_unused_layers no)
 			(net 46 "B6")
@@
 			(size 1.7526 1.7526)
 			(drill 1.0922)
-			(layers "*.Cu" "*.SilkS" "*.Mask")
+			(layers "*.Cu" "*.Mask")
 			(remove_unused_layers no)
 			(net 47 "B7")
@@
 			(size 1.7526 1.7526)
 			(drill 1.0922)
-			(layers "*.Cu" "*.SilkS" "*.Mask")
+			(layers "*.Cu" "*.Mask")
 			(remove_unused_layers no)
 			(net 48 "B8")
@@
 			(size 1.7526 1.7526)
 			(drill 1.0922)
-			(layers "*.Cu" "*.SilkS" "*.Mask")
+			(layers "*.Cu" "*.Mask")
 			(remove_unused_layers no)
 			(net 50 "B9")
@@
 			(size 1.7526 1.7526)
 			(drill 1.0922)
-			(layers "*.Cu" "*.SilkS" "*.Mask")
+			(layers "*.Cu" "*.Mask")
 			(remove_unused_layers no)
 			(net 54 "B10")
@@
 			(size 1.7526 1.7526)
 			(drill 1.0922)
-			(layers "*.Cu" "*.SilkS" "*.Mask")
+			(layers "*.Cu" "*.Mask")
 			(remove_unused_layers no)
 			(net 1 "B12")
@@
 			(size 1.7526 1.7526)
 			(drill 1.0922)
-			(layers "*.Cu" "*.SilkS" "*.Mask")
+			(layers "*.Cu" "*.Mask")
 			(remove_unused_layers no)
 			(net 3 "B13")
@@
 			(size 1.7526 1.7526)
 			(drill 1.0922)
-			(layers "*.Cu" "*.SilkS" "*.Mask")
+			(layers "*.Cu" "*.Mask")
 			(remove_unused_layers no)
 			(net 5 "B14")
@@
 			(size 1.7526 1.7526)
 			(drill 1.0922)
-			(layers "*.Cu" "*.SilkS" "*.Mask")
+			(layers "*.Cu" "*.Mask")
 			(remove_unused_layers no)
 			(net 7 "B15")
@@
 			(size 1.7526 1.7526)
 			(drill 1.0922)
-			(layers "*.Cu" "*.SilkS" "*.Mask")
+			(layers "*.Cu" "*.Mask")
 			(remove_unused_layers no)
 			(net 69 "C13")
@@
 			(size 1.7526 1.7526)
 			(drill 1.0922)
-			(layers "*.Cu" "*.SilkS" "*.Mask")
+			(layers "*.Cu" "*.Mask")
 			(remove_unused_layers no)
 			(net 68 "C14")
@@
 			(size 1.7526 1.7526)
 			(drill 1.0922)
-			(layers "*.Cu" "*.SilkS" "*.Mask")
+			(layers "*.Cu" "*.Mask")
 			(remove_unused_layers no)
 			(net 67 "C15")
@@
 			(size 1.7526 1.7526)
 			(drill 1.0922)
-			(layers "*.Cu" "*.SilkS" "*.Mask")
+			(layers "*.Cu" "*.Mask")
 			(remove_unused_layers no)
 			(net 70 "VBAT")
@@
 			(size 1.7526 1.7526)
 			(drill 1.0922)
-			(layers "*.Cu" "*.SilkS" "*.Mask")
+			(layers "*.Cu" "*.Mask")
 			(remove_unused_layers no)
 			(net 71 "X0")
@@
 			(size 1.7526 1.7526)
 			(drill 1.0922)
-			(layers "*.Cu" "*.SilkS" "*.Mask")
+			(layers "*.Cu" "*.Mask")
 			(remove_unused_layers no)
 			(net 72 "X1")
@@
 			(size 1.7526 1.7526)
 			(drill 1.0922)
-			(layers "*.Cu" "*.SilkS" "*.Mask")
+			(layers "*.Cu" "*.Mask")
 			(remove_unused_layers no)
 			(net 55 "X2")
@@
 			(size 1.7526 1.7526)
 			(drill 1.0922)
-			(layers "*.Cu" "*.SilkS" "*.Mask")
+			(layers "*.Cu" "*.Mask")
 			(remove_unused_layers no)
 			(net 66 "X3")
@@
 			(size 1.7526 1.7526)
 			(drill 1.0922)
-			(layers "*.Cu" "*.SilkS" "*.Mask")
+			(layers "*.Cu" "*.Mask")
 			(remove_unused_layers no)
 			(net 77 "b3V3")
@@
 			(size 1.7526 1.7526)
 			(drill 1.0922)
-			(layers "*.Cu" "*.SilkS" "*.Mask")
+			(layers "*.Cu" "*.Mask")
 			(remove_unused_layers no)
 			(net 75 "b5V")
@@
 			(size 1.7526 1.7526)
 			(drill 1.0922)
-			(layers "*.Cu" "*.SilkS" "*.Mask")
+			(layers "*.Cu" "*.Mask")
 			(remove_unused_layers no)
 			(net 76 "bG")
@@
 			(size 1.7526 1.7526)
 			(drill 1.0922)
-			(layers "*.Cu" "*.SilkS" "*.Mask")
+			(layers "*.Cu" "*.Mask")
 			(remove_unused_layers no)
 			(net 53 "t3V3")
@@
 			(size 1.7526 1.7526)
 			(drill 1.0922)
-			(layers "*.Cu" "*.SilkS" "*.Mask")
+			(layers "*.Cu" "*.Mask")
 			(remove_unused_layers no)
 			(net 51 "t5V")
@@
 			(size 1.7526 1.7526)
 			(drill 1.0922)
-			(layers "*.Cu" "*.SilkS" "*.Mask")
+			(layers "*.Cu" "*.Mask")
 			(remove_unused_layers no)
 			(net 52 "tG")
@@
 			(size 1.7526 1.7526)
 			(drill 1.0922)
-			(layers "*.Cu" "*.SilkS" "*.Mask")
+			(layers "*.Cu" "*.Mask")
 			(remove_unused_layers no)
 			(net 58 "A7")
@@
 			(size 1.7526 1.7526)
 			(drill 1.0922)
-			(layers "*.Cu" "*.SilkS" "*.Mask")
+			(layers "*.Cu" "*.Mask")
 			(remove_unused_layers no)
 			(net 57 "B0")
@@
 			(size 1.7526 1.7526)
 			(drill 1.0922)
-			(layers "*.Cu" "*.SilkS" "*.Mask")
+			(layers "*.Cu" "*.Mask")
 			(remove_unused_layers no)
 			(net 56 "B1")
@@
 			(size 1.7526 1.7526)
 			(drill 1.0922)
-			(layers "*.Cu" "*.SilkS" "*.Mask")
+			(layers "*.Cu" "*.Mask")
 			(remove_unused_layers no)
 			(net 54 "B10")
@@
 			(size 1.7526 1.7526)
 			(drill 1.0922)
-			(layers "*.Cu" "*.SilkS" "*.Mask")
+			(layers "*.Cu" "*.Mask")
 			(remove_unused_layers no)
 			(net 49 "B4")
@@
 			(size 1.7526 1.7526)
 			(drill 1.0922)
-			(layers "*.Cu" "*.SilkS" "*.Mask")
+			(layers "*.Cu" "*.Mask")
 			(remove_unused_layers no)
 			(net 45 "B5")
@@
 			(size 1.7526 1.7526)
 			(drill 1.0922)
-			(layers "*.Cu" "*.SilkS" "*.Mask")
+			(layers "*.Cu" "*.Mask")
 			(remove_unused_layers no)
 			(net 46 "B6")
@@
 			(size 1.7526 1.7526)
 			(drill 1.0922)
-			(layers "*.Cu" "*.SilkS" "*.Mask")
+			(layers "*.Cu" "*.Mask")
 			(remove_unused_layers no)
 			(net 47 "B7")
@@
 			(size 1.7526 1.7526)
 			(drill 1.0922)
-			(layers "*.Cu" "*.SilkS" "*.Mask")
+			(layers "*.Cu" "*.Mask")
 			(remove_unused_layers no)
 			(net 48 "B8")
@@
 			(size 1.7526 1.7526)
 			(drill 1.0922)
-			(layers "*.Cu" "*.SilkS" "*.Mask")
+			(layers "*.Cu" "*.Mask")
 			(remove_unused_layers no)
 			(net 50 "B9")
@@
 			(size 1.7526 1.7526)
 			(drill 1.0922)
-			(layers "*.Cu" "*.SilkS" "*.Mask")
+			(layers "*.Cu" "*.Mask")
 			(remove_unused_layers no)
 			(net 59 "A6")
@@
 			(size 1.7526 1.7526)
 			(drill 1.0922)
-			(layers "*.Cu" "*.SilkS" "*.Mask")
+			(layers "*.Cu" "*.Mask")
 			(remove_unused_layers no)
 			(net 60 "A5")
@@
 			(size 1.7526 1.7526)
 			(drill 1.0922)
-			(layers "*.Cu" "*.SilkS" "*.Mask")
+			(layers "*.Cu" "*.Mask")
 			(remove_unused_layers no)
 			(net 61 "A4")
@@
 			(size 1.7526 1.7526)
 			(drill 1.0922)
-			(layers "*.Cu" "*.SilkS" "*.Mask")
+			(layers "*.Cu" "*.Mask")
 			(remove_unused_layers no)
 			(net 62 "A3")
@@
 			(size 1.7526 1.7526)
 			(drill 1.0922)
-			(layers "*.Cu" "*.SilkS" "*.Mask")
+			(layers "*.Cu" "*.Mask")
 			(remove_unused_layers no)
 			(net 63 "A2")
@@
 			(size 1.7526 1.7526)
 			(drill 1.0922)
-			(layers "*.Cu" "*.SilkS" "*.Mask")
+			(layers "*.Cu" "*.Mask")
 			(remove_unused_layers no)
 			(net 64 "A1")
@@
 			(size 1.7526 1.7526)
 			(drill 1.0922)
-			(layers "*.Cu" "*.SilkS" "*.Mask")
+			(layers "*.Cu" "*.Mask")
 			(remove_unused_layers no)
 			(net 65 "A0")
@@
 			(size 1.7526 1.7526)
 			(drill 1.0922)
-			(layers "*.Cu" "*.SilkS" "*.Mask")
+			(layers "*.Cu" "*.Mask")
 			(remove_unused_layers no)
 			(net 67 "C15")
@@
 			(size 1.7526 1.7526)
 			(drill 1.0922)
-			(layers "*.Cu" "*.SilkS" "*.Mask")
+			(layers "*.Cu" "*.Mask")
 			(remove_unused_layers no)
 			(net 68 "C14")
@@
 			(size 1.7526 1.7526)
 			(drill 1.0922)
-			(layers "*.Cu" "*.SilkS" "*.Mask")
+			(layers "*.Cu" "*.Mask")
 			(remove_unused_layers no)
 			(net 69 "C13")
