File: split-tkl/output-left/pcbs/pcb-left.kicad_pcb (KiCad board)
At the start: 2 copper layers, 153.9 x 144.5 mm, 86 parts

Commit message: Renamed again
Parts:
- removed D36, D37: , ComboDiode
- removed MCU1: , Blackpill
- removed S36, S37: , MX
- moved D26 128.7 mm to (100.0, 81.2)
- moved S26 128.7 mm to (100.0, 76.2)
- moved D32 127.2 mm to (102.4, 181.2)
- moved D33 127.2 mm to (126.2, 181.2)
- moved S32 127.2 mm to (102.4, 176.2)
- moved S33 127.2 mm to (126.2, 176.2)
- moved D27 125.0 mm to (123.8, 81.2)
- moved S27 125.0 mm to (123.8, 76.2)
- moved D19 108.8 mm to (102.4, 162.2)
- moved S19 108.8 mm to (102.4, 157.2)
- moved D20 106.5 mm to (123.8, 162.2)
- moved S20 106.5 mm to (123.8, 157.2)
- moved D14 92.5 mm to (133.3, 143.1)
- moved S14 92.5 mm to (133.3, 138.1)
- moved D35 81.0 mm to (207.2, 181.2)
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Connections:
- D14 pad 1: B6 -> B7
- D14 pad 2: tab_y6 -> cap_q1
- D15 pad 2: cap_q1 -> cap_w2
- D16 pad 2: cap_w2 -> cap_e3
- D17 pad 2: cap_e3 -> cap_r4
- D18 pad 2: cap_r4 -> cap_t5
- D19 pad 1: B7 -> B8
- D19 pad 2: cap_t5 -> shift_lBord
- D20 pad 1: B7 -> B8
- D20 pad 2: cap_y6 -> shift_q1
- D21 pad 2: shift_lBord -> shift_w2
- D22 pad 2: shift_q1 -> shift_e3
- D23 pad 2: shift_w2 -> shift_r4
- D24 pad 2: shift_e3 -> shift_t5
- D25 pad 2: shift_r4 -> shift_y6
- D26 pad 1: B8 -> B4
- D26 pad 2: shift_t5 -> esc_only
- D27 pad 1: B8 -> B4
- D27 pad 2: shift_y6 -> f1_only
- D28 pad 2: esc_only -> f2_only
- D29 pad 2: f1_only -> f3_only
- D30 pad 2: f2_only -> f4_only
- D31 pad 2: f3_only -> f5_only
- D32 pad 1: B4 -> B9
- D32 pad 2: f4_only -> ctrl_only
- D33 pad 1: B4 -> B9
- D33 pad 2: f5_only -> win_only
- D34 pad 2: ctrl_only -> lAlt_only
- D35 pad 2: win_only -> space_only
- S14 pad 1: A10 -> B13
- S14 pad 2: tab_y6 -> cap_q1
- S15 pad 1: B13 -> B14
- S15 pad 2: cap_q1 -> cap_w2
- S16 pad 1: B14 -> B15
- S16 pad 2: cap_w2 -> cap_e3
- S17 pad 1: B15 -> A8
- S17 pad 2: cap_e3 -> cap_r4
- S18 pad 1: A8 -> A9
- S18 pad 2: cap_r4 -> cap_t5
- S19 pad 1: A9 -> B12
- S19 pad 2: cap_t5 -> shift_lBord
- S20 pad 1: A10 -> B13
- S20 pad 2: cap_y6 -> shift_q1
- S21 pad 1: B12 -> B14
- S21 pad 2: shift_lBord -> shift_w2
- S22 pad 1: B13 -> B15
- S22 pad 2: shift_q1 -> shift_e3
- S23 pad 1: B14 -> A8
- S23 pad 2: shift_w2 -> shift_r4
- S24 pad 1: B15 -> A9
- S24 pad 2: shift_e3 -> shift_t5
- S25 pad 1: A8 -> A10
- S25 pad 2: shift_r4 -> shift_y6
- S26 pad 1: A9 -> B12
- S26 pad 2: shift_t5 -> esc_only
- S27 pad 1: A10 -> B13
- S27 pad 2: shift_y6 -> f1_only
- S28 pad 1: B12 -> B14
- S28 pad 2: esc_only -> f2_only
- S29 pad 1: B13 -> B15
- S29 pad 2: f1_only -> f3_only
- S30 pad 1: B14 -> A8
- S30 pad 2: f2_only -> f4_only
- S31 pad 1: B15 -> A9
- S31 pad 2: f3_only -> f5_only
- S32 pad 1: A8 -> B12
- S32 pad 2: f4_only -> ctrl_only
- S33 pad 1: A9 -> B13
- S33 pad 2: f5_only -> win_only
- S34 pad 1: B12 -> B15
- S34 pad 2: ctrl_only -> lAlt_only
- S35 pad 1: B13 -> A9
- S35 pad 2: win_only -> space_only
Other:
- board size 153.9 x 144.5 mm -> 152.8 x 144.5 mm
